File: power.kicad_sch (KiCad schematic)
At the start: 23 parts, among them Q1 Si4948BEY, U2 171030601

Commit message: Test points TP1-TP5 in the schematic
TP1 +5V, TP2 GND, TP3 CAN_H, TP4 CAN_L (main sheet), TP5 VIN_PROT
(12 V after fuse and reverse polarity protection, power sheet).
Footprint TestPoint_Pad_D1.5mm (SMD). Not yet on the PCB (F8).

Co-Authored-By: Claude Opus 5.5 <noreply@anthropic.com>
Claude-Session: https://claude.ai/code/session_014h8cGi8SRWthYdGFH1Qgzz
Parts:
- added TP5: VIN_PROT, TestPoint:TestPoint_Pad_D1.5mm, symbol Connector:TestPoint
Connections:
- net VIN_PROT: now also TP5.1
Changed lines of the file:
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@@
+		)
+	)
+	(symbol
+		(lib_id "Connector:TestPoint")
+		(at 236.22 152.4 0)
+		(unit 1)
+		(body_style 1)
+		(exclude_from_sim no)
+		(in_bom yes)
+		(on_board yes)
+		(in_pos_files yes)
+		(dnp no)
+		(property "Reference" "TP5"
+			(at 236.22 159.258 0)
+			(show_name no)
+			(do_not_autoplace no)
+			(effects
+				(font
+					(size 1.27 1.27)
+				)
+			)
+		)
+		(property "Value" "VIN_PROT"
+			(at 236.22 157.48 0)
+			(show_name no)
+			(do_not_autoplace no)
+			(effects
+				(font
+					(size 1.27 1.27)
+				)
+			)
+		)
+		(property "Footprint" "TestPoint:TestPoint_Pad_D1.5mm"
+			(at 241.3 152.4 0)
+			(hide yes)
+			(show_name no)
+			(do_not_autoplace no)
+			(effects
+				(font
+					(size 1.27 1.27)
+				)
+			)
+		)
+		(property "Datasheet" ""
+			(at 241.3 152.4 0)
+			(hide yes)
+			(show_name no)
+			(do_not_autoplace no)
+			(effects
+				(font
+					(size 1.27 1.27)
+				)
+			)
+		)
+		(property "Description" "test point"
+			(at 236.22 152.4 0)
+			(hide yes)
+			(show_name no)
+			(do_not_autoplace no)
+			(effects
+				(font
+					(size 1.27 1.27)
+				)
+			)
+		)
+		(pin "1"
+		)
+		(instances
+			(project "JC8012P4A1C_I_W_Y_CAN"
+				(path "/3d717ebe-2c48-4d74-a932-f01128cae071/a2dcd761-dc69-4ab3-8065-aad2540c49d1"
+					(reference "TP5")
+					(unit 1)
+				)
+			)
+		)
+	)
+	(label "VIN_PROT"
+		(at 236.22 152.4 270)
+		(effects
+			(font
+				(size 1.27 1.27)
+			)
+			(justify right bottom)
 		)
 	)

Commit message: Input bulk capacitor: 2 x 22 uF/50 V (6.3 x 5.5) instead of 47 uF (8 x 6.5)
C9 and new C13: Wurth WCAP-ASLI 865080643008, 22 uF / 50 V, D6.3 x 5.5 mm,
in parallel on VIN_PROT. Lower than the old 8 x 6.5 mm part. A standard
electrolytic (not polymer) is kept on purpose: its ESR damps the input
filter (L2 + ceramic caps) and hot-plug ringing.
Footprint and 3D model from the Wurth KiCad library (rev26c).
Not yet on the PCB (F8).

Co-Authored-By: Claude Opus 5.5 <noreply@anthropic.com>
Claude-Session: https://claude.ai/code/session_014h8cGi8SRWthYdGFH1Qgzz
Parts:
- added C13: 22u/50V, JC8012P4A1C_CAN:CP_Wurth_WCAP-ASLI-D6.3L5.5, symbol Device:C_Polarized
- C9: value 47u/50V -> 22u/50V; footprint JC8012P4A1C_CAN:CP_Wurth_WCAP-ASLI-D8L6.5 -> JC8012P4A1C_CAN:CP_Wurth_WCAP-ASLI-D6.3L5.5; MPN 865080649013 -> 865080643008
Connections:
- net GND: now also C13.2
- net VIN_PROT: now also C13.1
Changed lines of the file:
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@@
 			)
 		)
-		(property "Value" "47u/50V"
+		(property "Value" "22u/50V"
 			(at 127.635 127 0)
 			(show_name no)
@@
 			)
 		)
-		(property "Footprint" "JC8012P4A1C_CAN:CP_Wurth_WCAP-ASLI-D8L6.5"
+		(property "Footprint" "JC8012P4A1C_CAN:CP_Wurth_WCAP-ASLI-D6.3L5.5"
 			(at 127.965 125.73 0)
 			(hide yes)
@@
 			)
 		)
-		(property "Datasheet" "https://www.we-online.com/catalog/datasheet/865080649013.pdf"
+		(property "Datasheet" "https://www.we-online.com/catalog/datasheet/865080643008.pdf"
 			(at 127 129.54 0)
 			(hide yes)
@@
 			)
 		)
-		(property "MPN" "865080649013"
+		(property "MPN" "865080643008"
 			(at 127 129.54 0)
 			(effects
@@
 				(path "/3d717ebe-2c48-4d74-a932-f01128cae071/a2dcd761-dc69-4ab3-8065-aad2540c49d1"
 					(reference "C9")
+					(unit 1)
+				)
+			)
+		)
+	)
+	(symbol
+		(lib_id "Device:C_Polarized")
+		(at 127 160.02 0)
+		(unit 1)
+		(body_style 1)
+		(exclude_from_sim no)
+		(in_bom yes)
+		(on_board yes)
+		(in_pos_files yes)
+		(dnp no)
+		(property "Reference" "C13"
+			(at 127.635 162.56 0)
+			(show_name no)
+			(do_not_autoplace no)
+			(effects
+				(font
+					(size 1.27 1.27)
+				)
+				(justify left)
+			)
+		)
+		(property "Value" "22u/50V"
+			(at 127.635 157.48 0)
+			(show_name no)
+			(do_not_autoplace no)
+			(effects
+				(font
+					(size 1.27 1.27)
+				)
+				(justify left)
+			)
+		)
+		(property "Footprint" "JC8012P4A1C_CAN:CP_Wurth_WCAP-ASLI-D6.3L5.5"
+			(at 127.965 156.21 0)
+			(hide yes)
+			(show_name no)
+			(do_not_autoplace no)
+			(effects
+				(font
+					(size 1.27 1.27)
+				)
+			)
+		)
+		(property "Datasheet" "https://www.we-online.com/catalog/datasheet/865080643008.pdf"
+			(at 127 160.02 0)
+			(hide yes)
+			(show_name no)
+			(do_not_autoplace no)
+			(effects
+				(font
+					(size 1.27 1.27)
+				)
+			)
+		)
+		(property "Description" "Polarized capacitor"
+			(at 127 160.02 0)
+			(hide yes)
+			(show_name no)
+			(do_not_autoplace no)
+			(effects
+				(font
+					(size 1.27 1.27)
+				)
+			)
+		)
+		(property "MPN" "865080643008"
+			(at 127 160.02 0)
+			(effects
+				(font
+					(size 1.27 1.27)
+				)
+				(hide yes)
+			)
+		)
+		(property "Manufacturer" "Wurth Elektronik"
+			(at 127 160.02 0)
+			(effects
+				(font
+					(size 1.27 1.27)
+				)
+				(hide yes)
+			)
+		)
+		(pin "1"
+		)
+		(pin "2"
+		)
+		(instances
+			(project "JC8012P4A1C_I_W_Y_CAN"
+				(path "/3d717ebe-2c48-4d74-a932-f01128cae071/a2dcd761-dc69-4ab3-8065-aad2540c49d1"
+					(reference "C13")
 					(unit 1)
 				)
@@
 		)
 	)
-)
+	(wire
+		(pts
+			(xy 127 156.21) (xy 127 153.67)
+		)
+		(stroke
+			(width 0)
+			(type default)
+		)
+	)
+	(label "VIN_PROT"
+		(at 127 153.67 90)
+		(effects
+			(font
+				(size 1.27 1.27)
+			)
+			(justify left bottom)
+		)
+	)
+	(wire
+		(pts
+			(xy 127 163.83) (xy 127 166.37)
+		)
+		(stroke
+			(width 0)
+			(type default)
+		)
+	)
+	(global_label "GND"
+		(shape passive)
+		(at 127 166.37 270)
+		(effects
+			(font
+				(size 1.27 1.27)
+			)
+			(justify right bottom)
+		)
+	))

Commit message: Test points excluded from BOM, README: hand assembly, stencil, BOM export
Co-Authored-By: Claude Opus 5.5 <noreply@anthropic.com>
Claude-Session: https://claude.ai/code/session_014h8cGi8SRWthYdGFH1Qgzz
Parts:
- TP5: now left out of the parts list
Changed lines of the file:
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@@
 		(body_style 1)
 		(exclude_from_sim no)
-		(in_bom yes)
+		(in_bom no)
 		(on_board yes)
 		(in_pos_files yes)
