File: JC8012P4A1C_I_W_Y_CAN.kicad_pcb (KiCad board)
At the start: 6 copper layers, 66 x 54 mm, 39 parts, among them J1 610110249121, J2 68711414522, J3 653104131822, Q1 Si4948BEY, U1 TLE9250VSJ, U2 171030601

Commit message: Board marking, 3D images, README: PCB and manufacturing
- Silkscreen: project name, Rev A 2026-10; "cut" mark at J1 pin 10
- docs/: 3D renders (top and isometric) from kicad-cli pcb render
- README: layer stack, via-in-pad (epoxy filled and capped), stitching,
  how to generate Gerber and drill files
- production/ (generated outputs) ignored

Co-Authored-By: Claude Opus 5.5 <noreply@anthropic.com>
Claude-Session: https://claude.ai/code/session_014h8cGi8SRWthYdGFH1Qgzz
Other:
- board text added: "I_W_Y_CAN"
- board text added: "JC8012P4A1C"
- board text added: "Rev A 2026-10"
- board text added: "cut"
Changed lines of the file:
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@@
 		(layer "Edge.Cuts")
+	)
+	(gr_text "cut"
+		(at 116.3 144.58 0)
+		(layer "F.SilkS")
+		(effects
+			(font
+				(size 0.8 0.8)
+				(thickness 0.15)
+			)
+		)
+	)
+	(gr_text "JC8012P4A1C"
+		(at 148.5 134 0)
+		(layer "F.SilkS")
+		(effects
+			(font
+				(size 1 1)
+				(thickness 0.15)
+			)
+		)
+	)
+	(gr_text "I_W_Y_CAN"
+		(at 148.5 135.8 0)
+		(layer "F.SilkS")
+		(effects
+			(font
+				(size 1 1)
+				(thickness 0.15)
+			)
+		)
+	)
+	(gr_text "Rev A  2026-10"
+		(at 148.5 137.6 0)
+		(layer "F.SilkS")
+		(effects
+			(font
+				(size 1 1)
+				(thickness 0.15)
+			)
+		)
 	)
 	(segment

Commit message: PCB: C9/C13 2 x 22 uF and test points TP1-TP5 placed and connected
- C9 and C13 (6.3 x 5.5) stacked in the former C9 column, + towards the
  VIN_PROT side, kept out of the FFC path above J2. C13 + connected to
  C9 + with a 0.8 mm trace, two GND vias in each GND pad
- TP1 +5V / TP2 GND next to J3 (TP1 with +5V via in pad), TP3 CAN_H /
  TP4 CAN_L on the CAN lines between D1 and J1, TP5 in the VIN_PROT pour
- Test points show the net name on the silkscreen instead of TPx
- Silkscreen texts re-placed (C9, C13, D1, "cut")
- 3D images and README (test points) updated
DRC: 0 violations, 0 unconnected, schematic parity OK.

Co-Authored-By: Claude Opus 5.5 <noreply@anthropic.com>
Claude-Session: https://claude.ai/code/session_014h8cGi8SRWthYdGFH1Qgzz
Parts:
- added C13: 22u/50V, JC8012P4A1C_CAN:CP_Wurth_WCAP-ASLI-D6.3L5.5, F.Cu at (125.5, 107.9)
- added TP1: +5V, TestPoint:TestPoint_Pad_D1.5mm, F.Cu at (155.5, 142.0)
- added TP2: GND, TestPoint:TestPoint_Pad_D1.5mm, F.Cu at (155.5, 144.5)
- added TP3: CAN_H, TestPoint:TestPoint_Pad_D1.5mm, F.Cu at (115.3, 147.6)
- added TP4: CAN_L, TestPoint:TestPoint_Pad_D1.5mm, F.Cu at (113.0, 152.6)
- added TP5: VIN_PROT, TestPoint:TestPoint_Pad_D1.5mm, F.Cu at (129.0, 121.0)
- C9: value 47u/50V -> 22u/50V; footprint JC8012P4A1C_CAN:CP_Wurth_WCAP-ASLI-D8L6.5 -> JC8012P4A1C_CAN:CP_Wurth_WCAP-ASLI-D6.3L5.5
- moved C9 1.25 mm to (125.5, 115.8), turned to 180 degrees
Routing:
- net /Versorgung/VIN_PROT: track 32.4 -> 40.3 mm
- net /CAN_H: track 31.0 -> 33.4 mm
- net /CAN_L: track 35.2 -> 37.2 mm
- net GND: vias 267 -> 266
- net +5V: vias 15 -> 16

Commit message: Mounting holes H1-H4 replaced by SMD steel spacers Wurth 9774025943R (2.5 mm, M2x6)
Co-Authored-By: Claude Opus 5.5 <noreply@anthropic.com>
Claude-Session: https://claude.ai/code/session_014h8cGi8SRWthYdGFH1Qgzz
Parts:
- H1, H2, H3, H4: value M2 -> Spacer M2 L2.5; footprint MountingHole:MountingHole_2.2mm_M2_Pad_Via -> JC8012P4A1C_CAN:A_Wurth_WA-SMST_9774025943R
